File: 8088_sbc2.sch (KiCad schematic (older format))
At the start: 4 parts

Commit message: working on schematic
Parts:
- added C? (x2): 100n, symbol C
- added R? (x3): 10k, symbol R
- added SW?: SW_PUSH, symbol SW_PUSH
- added U?: TL770xA, symbol TL770xA
- added U?: OSC_SMALL, symbol OSC_SMALL
- added U? (x2): 74HC138, symbol 74HC138
Connections:
- net labels added: CLK, IO/nM, IODEV0_EN, IODEV1_EN, nRES
- wire segments 36 -> 86
- no-connect marks 0 -> 11
Other:
- note added: "Address decoder for IO\n"
- note added: "Address decoder for MEM\n"

Commit message: am schaltplan weitergearbeitet
Parts:
- added RR?: RR8, symbol RR8
- added U? (x2): 74HC573, symbol 74HC573
- added U?: 10xLEDBAR, symbol 10xLEDBAR
- added U?: 74HC14_OWN, symbol 74HC14_OWN
- added U?: 74HC08, symbol 74HC08
- added U?: 74HC32, symbol 74HC32
Connections:
- net labels added: INTR, IODEV0_WREN, NMI, S3, S4, S5, S6, nFRAMEN, nIODEV0_EN, nIODEV0_WREN, nIODEV1_EN, nRAMEN, nRAMHIEN, nRAMLOEN, nRD, nROMEN, nWR
- net labels removed: IODEV0_EN, IODEV1_EN
- wire segments 86 -> 151
- no-connect marks 11 -> 23

Commit message: schematic erc good.
Parts:
- added 1K1: R, symbol R
- added C1, C10, C11, C12, C13, C14, C15, C16, C19, C2, C20, C21, C22, C4, C6, C9: 100n, symbol C
- added C17, C18: 4u7, symbol C
- added F1: FUSE, symbol FUSE
- added L1: INDUCTOR, symbol INDUCTOR
- added P1: CONN_02X10, symbol CONN_02X10
- added P2: JMP_USB_PWR, symbol CONN_01X02
- added P3: USB_B, symbol USB_B
- added P_GND1: GND, symbol CONN_01X02
- added P_VCC1: VCC, symbol CONN_01X02
- added Q1: IRLML6402, symbol Q_PMOS_GSD
- added R4, R5: 10k, symbol R
- added RR1: 8x300R, symbol RR8
- added SW2, SW3, SW4, SW5, SW6, SW7, SW8, SW9: SWITCH_INV, symbol SWITCH_INV
- added U13: 28C64, symbol 28C64
- added U14: AS6C4008, symbol AS6C4008
- added U15: 16C550, symbol 16C550
- added U16: FM1808B, symbol FM1808B
- added U17: FT232RL, symbol FT232RL
- added U8: 74HC573, symbol 74HC573
- RR2: renamed from RR?; value RR8 -> 8x10K
- gave numbers to parts that had none: 20
Connections:
- net labels added: IN0, IN1, IN2, IN3, IN4, IN5, IN6, IN7, OUT0, OUT1, OUT2, OUT3, OUT4, OUT5, OUT6, OUT7, RES, nIODEV0_RDEN
- wire segments 151 -> 406
- no-connect marks 23 -> 55
Other:
- moved on the sheet: RR2, U12, U18

Commit message: looks good :D
Parts:
- removed C16, C22: 100n, symbol C
- removed C17, C18: 4u7, symbol C
- removed R4, R5: 10k, symbol R
- removed U16: FM1808B, symbol FM1808B
- added C10: 4u7, Capacitors_ThroughHole:C_Radial_D6.3_L11.2_P2.5, symbol CP1
- added C20: 4u7, Capacitors_ThroughHole:C_Radial_D7.5_L11.2_P2.5, symbol CP1
- added C7: 100n, Capacitors_ThroughHole:C_Disc_D3_P2.5, symbol C
- C1: renamed from C5; footprint (none) -> Capacitors_ThroughHole:C_Disc_D3_P2.5
- C11: renamed from C2; footprint (none) -> Capacitors_ThroughHole:C_Disc_D3_P2.5
- C12: renamed from C3; footprint (none) -> Capacitors_ThroughHole:C_Disc_D3_P2.5
- C13: renamed from C6; footprint (none) -> Capacitors_ThroughHole:C_Disc_D3_P2.5
- C14: renamed from C9; footprint (none) -> Capacitors_ThroughHole:C_Disc_D3_P2.5
- C15: renamed from C1; footprint (none) -> Capacitors_ThroughHole:C_Disc_D3_P2.5
- C16: renamed from C10; footprint (none) -> Capacitors_ThroughHole:C_Disc_D3_P2.5
- C17: renamed from C11; footprint (none) -> Capacitors_ThroughHole:C_Disc_D3_P2.5
- C18: renamed from C4; footprint (none) -> Capacitors_ThroughHole:C_Disc_D3_P2.5
- C19: renamed from C12; footprint (none) -> Capacitors_ThroughHole:C_Disc_D3_P2.5
- C2: renamed from C15; footprint (none) -> Capacitors_ThroughHole:C_Disc_D3_P2.5
- C21: renamed from C19; footprint (none) -> Capacitors_ThroughHole:C_Disc_D3_P2.5
- C3: renamed from C20; footprint (none) -> Capacitors_ThroughHole:C_Disc_D3_P2.5
- C4: renamed from C7; footprint (none) -> Capacitors_ThroughHole:C_Disc_D3_P2.5
- C5: renamed from C21; footprint (none) -> Capacitors_ThroughHole:C_Disc_D3_P2.5
- C6: renamed from C14; footprint (none) -> Capacitors_ThroughHole:C_Disc_D3_P2.5
- C8: footprint (none) -> Capacitors_ThroughHole:C_Disc_D3_P2.5
- C9: renamed from C13; footprint (none) -> Capacitors_ThroughHole:C_Disc_D3_P2.5
- F1: footprint (none) -> Capacitors_SMD:C_1206_HandSoldering
- GND1: renamed from P_GND1; footprint (none) -> Pin_Headers:Pin_Header_Straight_1x02
- I0: renamed from SW2; footprint (none) -> 8088_sbc2:EG1218
- I1: renamed from SW3; footprint (none) -> 8088_sbc2:EG1218
- I2: renamed from SW4; footprint (none) -> 8088_sbc2:EG1218
- I3: renamed from SW5; footprint (none) -> 8088_sbc2:EG1218
- I4: renamed from SW6; footprint (none) -> 8088_sbc2:EG1218
- I5: renamed from SW7; footprint (none) -> 8088_sbc2:EG1218
- I6: renamed from SW8; footprint (none) -> 8088_sbc2:EG1218
- I7: renamed from SW9; footprint (none) -> 8088_sbc2:EG1218
- L1: footprint (none) -> Capacitors_SMD:C_0805_HandSoldering
- P1: footprint (none) -> Pin_Headers:Pin_Header_Straight_2x10
- P2: footprint (none) -> Pin_Headers:Pin_Header_Straight_1x02
- P3: footprint (none) -> Connect:USB_B
- Q1: footprint (none) -> TO_SOT_Packages_SMD:SOT-23_Handsoldering
- R1, R2, R3: footprint (none) -> Resistors_ThroughHole:Resistor_Horizontal_RM7mm
- R4: renamed from 1K1; value R -> 1K; footprint (none) -> Resistors_SMD:R_0805_HandSoldering
- RR1, RR2: footprint (none) -> Pin_Headers:Pin_Header_Straight_1x09
- SW1: footprint (none) -> Buttons_Switches_ThroughHole:SW_PUSH_6mm
- U1: renamed from U3; footprint (none) -> Housings_DIP:DIP-40_W15.24mm
- U11: renamed from U4; footprint (none) -> Housings_DIP:DIP-20_W7.62mm
- U12: renamed from U5; footprint (none) -> Housings_DIP:DIP-20_W7.62mm
- U13: renamed from U6; footprint (none) -> Housings_DIP:DIP-20_W7.62mm
- U14: renamed from U8; footprint (none) -> Housings_DIP:DIP-20_W7.62mm
- U15: renamed from U2; footprint (none) -> Housings_DIP:DIP-16_W7.62mm
- U16: renamed from U9; footprint (none) -> Housings_DIP:DIP-16_W7.62mm
- U17: renamed from U12; footprint (none) -> Housings_DIP:DIP-14_W7.62mm
- U18: renamed from U1; footprint (none) -> Housings_DIP:DIP-14_W7.62mm
- U19: renamed from U11; footprint (none) -> Housings_DIP:DIP-14_W7.62mm
- U2: renamed from U13; footprint (none) -> Housings_DIP:DIP-28_W15.24mm
- U20: renamed from U7; footprint (none) -> Housings_DIP:DIP-20_W7.62mm
- U3: renamed from U14; footprint (none) -> Housings_DIP:DIP-32_W15.24mm
- U4: renamed from U10; footprint (none) -> Housings_DIP:DIP-8_W7.62mm
- U5: renamed from U15; footprint (none) -> Housings_DIP:DIP-40_W15.24mm
- U6: renamed from U17; footprint (none) -> Housings_SSOP:SSOP-28_5.3x10.2mm_Pitch0.65mm
- U7: renamed from U18; footprint (none) -> Housings_DIP:DIP-8_W7.62mm
- VCC1: renamed from P_VCC1; footprint (none) -> Pin_Headers:Pin_Header_Straight_1x02
Connections:
- wire segments 406 -> 375
Other:
- moved on the sheet: U13

Commit message: DRC and ERC OK. making some gerbers now?!
Connections:
- net nFRAMEN: no longer names the net of U15.13 (nY2)
- no-connect marks 55 -> 56
Changed lines of the file:
@@
 	1    0    0    -1
 $EndComp
-Text Label 8350 1450 0    60   ~ 0
-nFRAMEN
 Text Label 8350 1350 0    60   ~ 0
 nRAMHIEN
@@
 Wire Wire Line
 	8200 1550 8350 1550
-Wire Wire Line
-	8200 1450 8350 1450
 Connection ~ 6450 1850
 Wire Wire Line
@@
 Wire Wire Line
 	10600 3450 10600 2900
+NoConn ~ 8200 1450
 $EndSCHEMATC
